File: Ematch_board/Mainboard.kicad_pcb (KiCad board)
At the start: 4 copper layers, 57.3 x 53.3 mm, 125 parts, among them J1 Conn_01x02_Male, J10 Conn_01x02_Male, J11 Conn_Coaxial, J2 Conn_01x02_Male, J3 Conn_01x02_Male, J4 Conn_01x02_Male, J5 Conn_01x02_Male, J6 Conn_01x02_Male, J7 RBUS, J8 USB_C_Receptacle_USB2.0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

Commit message: Added flint and steel name and picture
Parts:
- added G***: LOGO, LOGO, B.Cu at (152.6, 93.2)
Other:
- board text added: "FLINT AND STEEL"
Changed lines of the file:
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@@
     )
   )
+  (footprint "LOGO" (layer "B.Cu")
+    (at 152.568069 93.171932 180)
+    (attr board_only exclude_from_pos_files exclude_from_bom)
+    (fp_text reference "G***" (at 0 0) (layer "B.SilkS") hide
+      (effects (font (size 1.524 1.524) (thickness 0.3)) (justify mirror))
+    )
+    (fp_text value "LOGO" (at 0.75 0) (layer "B.SilkS") hide
+      (effects (font (size 1.524 1.524) (thickness 0.3)) (justify mirror))
+    )
+    (fp_poly (pts
+        (xy -1.876136 11.256818)
+        (xy -1.876136 9.380681)
+        (xy -3.752272 9.380681)
+        (xy -3.752272 7.504545)
+        (xy -5.628409 7.504545)
+        (xy -5.628409 0)
+        (xy -3.752272 0)
+        (xy -3.752272 1.876136)
+        (xy 0 1.876136)
+        (xy 0 -1.876137)
+        (xy -1.876136 -1.876137)
+        (xy -1.876136 -3.752273)
+        (xy -3.752272 -3.752273)
+        (xy -3.752272 -5.62841)
+        (xy -7.504545 -5.62841)
+        (xy -7.504545 -3.752273)
+        (xy -9.380681 -3.752273)
+        (xy -9.380681 -1.876137)
+        (xy -7.504545 -1.876137)
+        (xy -7.504545 -3.752273)
+        (xy -3.752272 -3.752273)
+        (xy -3.752272 -1.876137)
+        (xy -1.876136 -1.876137)
+        (xy -1.876136 0)
+        (xy -3.752272 0)
+        (xy -3.752272 -1.876137)
+        (xy -5.628409 -1.876137)
+        (xy -5.628409 0)
+        (xy -7.504545 0)
+        (xy -7.504545 7.504545)
+        (xy -5.628409 7.504545)
+        (xy -5.628409 9.380681)
+        (xy -3.752272 9.380681)
+        (xy -3.752272 11.256818)
+        (xy -7.504545 11.256818)
+        (xy -7.504545 9.380681)
+        (xy -9.380681 9.380681)
+        (xy -9.380681 -1.876137)
+        (xy -11.256818 -1.876137)
+        (xy -11.256818 9.380681)
+        (xy -9.380681 9.380681)
+        (xy -9.380681 11.256818)
+        (xy -7.504545 11.256818)
+        (xy -7.504545 13.132954)
+        (xy -3.752272 13.132954)
+        (xy -3.752272 11.256818)
+      ) (layer "B.SilkS") (width 0) (fill solid))
+    (fp_poly (pts
+        (xy 0 5.628409)
+        (xy -3.752272 5.628409)
+        (xy -3.752272 7.504545)
+        (xy -1.876136 7.504545)
+        (xy -1.876136 9.380681)
+        (xy 0 9.380681)
+      ) (layer "B.SilkS") (width 0) (fill solid))
+    (fp_poly (pts
+        (xy 9.380682 0)
+        (xy 9.380682 -3.752273)
+        (xy 11.256819 -3.752273)
+        (xy 11.256819 -7.504546)
+        (xy 13.132955 -7.504546)
+        (xy 13.132955 -11.256819)
+        (xy 11.256819 -11.256819)
+        (xy 11.256819 -13.132955)
+        (xy 5.62841 -13.132955)
+        (xy 5.62841 -15.009091)
+        (xy 1.876137 -15.009091)
+        (xy 1.876137 -13.132955)
+        (xy 0 -13.132955)
+        (xy 0 -11.256819)
+        (xy -1.876136 -11.256819)
+        (xy -1.876136 -9.380682)
+        (xy 0 -9.380682)
+        (xy 1.876137 -9.380682)
+        (xy 1.876137 -7.504546)
+        (xy 3.752273 -7.504546)
+        (xy 3.752273 -5.62841)
+        (xy 5.62841 -5.62841)
+        (xy 5.62841 -3.752273)
+        (xy 7.504546 -3.752273)
+        (xy 7.504546 0)
+        (xy 5.62841 0)
+        (xy 5.62841 -1.876137)
+        (xy 3.752273 -1.876137)
+        (xy 3.752273 -3.752273)
+        (xy 1.876137 -3.752273)
+        (xy 1.876137 -5.62841)
+        (xy 0 -5.62841)
+        (xy 0 -9.380682)
+        (xy -1.876136 -9.380682)
+        (xy -1.876136 -5.62841)
+        (xy 0 -5.62841)
+        (xy 0 -3.752273)
+        (xy 1.876137 -3.752273)
+        (xy 1.876137 -1.876137)
+        (xy 3.752273 -1.876137)
+        (xy 3.752273 0)
+        (xy 5.62841 0)
+        (xy 5.62841 1.876136)
+        (xy 7.504546 1.876136)
+        (xy 7.504546 0)
+      ) (layer "B.SilkS") (width 0) (fill solid))
+  )
   (gr_rect locked (start 117.968 69.5047) (end 175.2248 122.8067) (layer "Edge.Cuts") (width 0.05) (fill none))
+  (gr_text "FLINT AND STEEL" (at 147.83 76.51) (layer "B.SilkS")
+    (effects (font (size 3.5 3.5) (thickness 0.6)) (justify mirror))
+  )
   (gr_text "5V_TP\n" (at 166.68 120.62 90) (layer "F.SilkS")
     (effects (font (size 0.8 0.8) (thickness 0.1)))

Commit message: Added writepad and iclr logo to back silkscreen
Parts:
- added G***: LOGO, iclr:iclr_logo, B.Cu at (128.5, 94.3)
- moved G*** 3.21 mm to (154.6, 95.7)
Other:
- board text added: "FLINT & STEEL"
- board text removed: "FLINT AND STEEL"
