File: Hardware/flintandsteel.kicad_pcb (KiCad board)
At the start: 4 copper layers, 44 x 62.9 mm, 143 parts, among them J1 RBUS, J2 USB_C_Receptacle_USB2.0, J3 Conn_01x02_Male, J4 Conn_01x02_Male, J5 Conn_01x02_Male, J6 Conn_01x02_Male, Q1 NCV8403, Q2 NCV8403, Q3 NCV8403, Q4 NCV8403, U1 ESP32-S3, U2 SN65HVD230, U3 LM66200DRLR, U4 MAX77827AEFD+T, U5 SC4215, U6 LTV-247, U7 SiC431, Y1 40MHz±10ppm

Commit message: finished? (pre-review)
Parts:
- removed C43, C47, C49: DNP, Capacitor_SMD:C_1206_3216Metric
- removed TP3: TestPoint, TestPoint:TestPoint_Pad_D1.0mm
- removed TP4, TP5, TP7: TestPoint, TestPoint:TestPoint_Pad_D1.5mm
- added G***: LOGO, LOGO, B.Cu at (67.0, 94.3)
- added G***: LOGO, iclr:iclr_logo_estd2018_10mm, B.Cu at (74.8, 110.1)
- added R37: 1.5k, Resistor_SMD:R_0402_1005Metric, F.Cu at (57.1, 96.7)
- added R38: 2.2k, Resistor_SMD:R_0402_1005Metric, F.Cu at (58.0, 96.7)
- TP1: renamed from TP2; moved to B.Cu
- TP10, TP9: moved to B.Cu
- TP2: renamed from TP1; moved to B.Cu
- TP6, TP8: footprint TestPoint:TestPoint_Pad_D1.5mm -> TestPoint:TestPoint_Pad_D1.0mm
- TXLED1, USBLED1: footprint Resistor_SMD:R_0402_1005Metric -> Diode_SMD:D_0402_1005Metric
- moved TP8 158.8 mm to (54.2, 79.3)
- moved USBLED1 158.0 mm to (50.5, 70.7), turned to 90 degrees
- moved TP6 157.9 mm to (54.2, 77.9)
- moved R13 156.7 mm to (51.4, 70.7), turned to 90 degrees
- moved TP2 147.7 mm to (55.4, 77.5), turned to -90 degrees
- moved TP1 146.0 mm to (57.4, 78.8), turned to -90 degrees
- moved TXLED1 144.8 mm to (61.0, 81.5), turned to 180 degrees
- moved C1 142.0 mm to (50.0, 89.3), turned to -90 degrees
- moved L1 141.8 mm to (51.8, 87.5), turned to 90 degrees
- moved C6 141.2 mm to (52.8, 87.4), turned to -90 degrees
- moved C4 140.7 mm to (50.9, 89.3), turned to -90 degrees
- moved C5 139.1 mm to (51.8, 89.3), turned to -90 degrees
- moved R6 137.7 mm to (61.0, 82.5), turned to 180 degrees
- moved TP10 133.0 mm to (58.2, 85.0), turned to 90 degrees
- moved R4 130.9 mm to (57.3, 94.4)
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- renumbered D7 to D4, D4 to D7
Connections:
- BOOTJUMPER1 pad 1: /BOOT -> GND
- BOOTJUMPER1 pad 2: GND -> /BOOT
- ENJUMPER1 pad 1: /CHIP_PU -> GND
- ENJUMPER1 pad 2: GND -> /CHIP_PU
- Firing2 pad 2: /Nuke 3 -> /Nuke 2
- Firing3 pad 2: /Nuke 2 -> /Nuke 3
- Q2 pad 1: /Nuke 3 -> /Nuke 2
- Q3 pad 1: /Nuke 2 -> /Nuke 3
- R21 pad 1: /Cont 3 -> /Cont 2
- R26 pad 1: /Cont 2 -> /Cont 3
- TP1 pad 1: /Data+ -> /Data-
- TP2 pad 1: /Data- -> /Data+
- U1 pad 15: unconnected-(U1-GPIO10/ADC1_CH9-Pad15) -> /BuckPGOOD
- U1 pad 23: unconnected-(U1-GPIO17/ADC2_CH6/DAC_2-Pad23) -> /CAN_RX
- U1 pad 24: unconnected-(U1-GPIO18/ADC2_CH7/DAC_1-Pad24) -> /CAN_TX
- U1 pad 27: unconnected-(U1-GPIO21-Pad27) -> /Nuke 4
- U1 pad 37: unconnected-(U1-SPICLK_P/GPIO47-Pad37) -> /Cont 2
- U1 pad 38: unconnected-(U1-GPIO33-Pad38) -> /Nuke 3
- U1 pad 39: unconnected-(U1-GPIO34-Pad39) -> /Nuke 2
- U1 pad 40: unconnected-(U1-GPIO35-Pad40) -> /Nuke 1
- U1 pad 41: unconnected-(U1-GPIO36-Pad41) -> /Cont 1
- U1 pad 42: unconnected-(U1-GPIO37-Pad42) -> /Cont 4
- U1 pad 43: unconnected-(U1-GPIO38-Pad43) -> /Cont 3
- U6 pad 11: /Cont 2 -> /Cont 3
- U6 pad 13: /Cont 3 -> /Cont 2
Routing:
- net /Data+: track 0.00 -> 32.3 mm, vias 0 -> 2
- net VBUS: track 5.27 -> 35.8 mm, vias 2 -> 4
- net /Data-: track 0.00 -> 29.8 mm, vias 0 -> 2
- net +3V3: track 10.4 -> 36.6 mm, vias 5 -> 13
- net /Nuke 4: track 0.00 -> 23.4 mm
- net /buckC/PGOOD: track 0.00 -> 22.5 mm, vias 0 -> 3
- net /Cont 4: track 0.00 -> 21.8 mm
- net /CAN+: track 9.08 -> 29.0 mm
- net /CAN-: track 8.88 -> 28.2 mm
- net /Cont 3: track 0.00 -> 18.0 mm, vias 0 -> 2
- net /Nuke 3: track 0.00 -> 17.7 mm
- net /Cont 2: track 0.00 -> 17.2 mm, vias 0 -> 2
- net RBUS_uC_V: track 0.00 -> 15.8 mm
- net /CHIP_PU: track 0.00 -> 13.7 mm
- net /BOOT: track 0.00 -> 13.3 mm
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- added copper zone on In2.Cu, net +3V3
Other:
- board size 44 x 62.9 mm -> 44 x 63 mm
- rule pad_to_mask_clearance: 0.05 -> 0
- board text added: "Batch Number - JLCJLCJLCJLC"
- board text added: "locked"
