File: Hardware/flintandsteel.kicad_pcb (KiCad board)
At the start: 4 copper layers, 44 x 58 mm, 143 parts, among them J1 RBUS, J2 USB_C_Receptacle_USB2.0, J3 Conn_01x02_Male, J4 Conn_01x02_Male, J5 Conn_01x02_Male, J6 Conn_01x02_Male, Q1 BSZ025N04LS, Q2 BSZ025N04LS, Q3 BSZ025N04LS, Q4 BSZ025N04LS, Q5 BSZ025N04LS, Q6 BSZ025N04LS, U1 ESP32-S3, U2 SN65HVD230, U3 LM66200DRLR, U4 MAX77827AEFD+T, U5 SC4215, U6 LTV-247, U7 INA219AxDCN, U8 LM74810, Y1 R940000171

Commit message: files
Parts:
- added D20: RCLAMP3346PQTNT, iclr:RCLAMP3346PQTNT, F.Cu at (116.4, 93.2)
- added J7: 1723103102, iclr:CONN_1723102000_02_MOL, F.Cu at (144.3, 93.3)
- added R41: 10k, Resistor_SMD:R_0402_1005Metric, B.Cu at (108.8, 94.8)
- added R42: 10k, Resistor_SMD:R_0402_1005Metric, B.Cu at (109.8, 94.8)
- added R43: 10k, Resistor_SMD:R_0402_1005Metric, B.Cu at (113.8, 94.8)
- added R44: 10k, Resistor_SMD:R_0402_1005Metric, B.Cu at (114.8, 94.8)
- added R45: 10k, Resistor_SMD:R_0402_1005Metric, B.Cu at (111.5, 101.2)
- added R46: 10k, Resistor_SMD:R_0402_1005Metric, B.Cu at (109.6, 101.2)
- added R47: 10k, Resistor_SMD:R_0402_1005Metric, F.Cu at (136.2, 118.6)
- H4: footprint MountingHole:MountingHole_3.2mm_M3_DIN965 -> MountingHole:MountingHole_3.2mm_M3_DIN965_Pad
- J3, J4, J5: value Conn_01x02_Male -> 1723103102; footprint TerminalBlock_Phoenix:TerminalBlock_Phoenix_PT-1,5-2-3.5-H_1x02_P3.50mm_Horizontal -> iclr:CONN_1723102000_02_MOL
- J6: value Conn_01x02_Male -> GPIO Breakout; footprint TerminalBlock_Phoenix:TerminalBlock_Phoenix_PT-1,5-2-3.5-H_1x02_P3.50mm_Horizontal -> Connector_PinSocket_2.54mm:PinSocket_2x04_P2.54mm_Vertical
- R37, R38, R39: moved to F.Cu
- moved J6 33.5 mm to (115.6, 99.3), turned to -90 degrees
- moved J5 12.5 mm to (144.3, 116.5)
- moved J4 10.4 mm to (144.3, 104.9)
- moved D1 8.64 mm to (118.8, 106.5), turned to 0 degrees
- moved R9 6.67 mm to (121.3, 107.9), turned to 0 degrees
- moved C17 6.42 mm to (121.7, 106.5), turned to 180 degrees
- moved J1 6.10 mm to (109.0, 117.0)
- moved D19 6.04 mm to (120.1, 111.9), turned to 0 degrees
- moved R31 5.29 mm to (124.4, 113.7), turned to 45 degrees
- moved C29 5.02 mm to (118.6, 115.1)
- moved R35 4.88 mm to (134.1, 119.7)
- moved TP4 4.75 mm to (123.7, 112.2)
- moved C1 4.71 mm to (112.8, 87.2), turned to -90 degrees
- moved R5 4.68 mm to (122.6, 114.8)
- moved R39 4.63 mm to (121.5, 112.0), turned to -90 degrees
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Connections:
- J4 pad 2: Net-(D15-A) -> Net-(D17-A)
- J5 pad 2: Net-(D17-A) -> Net-(D18-A)
- J6 pad 1: /PyroPWR -> GND
- J6 pad 2: Net-(D18-A) -> /GPIO5
- U1 pad 10: unconnected-(U1-GPIO5/ADC1_CH4-Pad10) -> /GPIO5
- U1 pad 11: unconnected-(U1-GPIO6/ADC1_CH5-Pad11) -> /GPIO6
- U1 pad 12: unconnected-(U1-GPIO7/ADC1_CH6-Pad12) -> /GPIO7
- U1 pad 6: unconnected-(U1-GPIO1/ADC1_CH0-Pad6) -> /GPIO1
- U1 pad 7: unconnected-(U1-GPIO2/ADC1_CH1-Pad7) -> /GPIO2
- U1 pad 9: unconnected-(U1-GPIO4/ADC1_CH3-Pad9) -> /GPIO4
Routing:
- net /GPIO7: track 0.00 -> 25.0 mm
- net /GPIO6: track 0.00 -> 19.0 mm
- net /GPIO1: track 0.00 -> 18.5 mm
- net /GPIO2: track 0.00 -> 16.2 mm
- net /CAN-: track 28.3 -> 12.5 mm
- net /GPIO4: track 0.00 -> 13.4 mm
- net /CAN+: track 29.1 -> 17.1 mm
- net /GPIO5: track 0.00 -> 11.4 mm
- net RBUS_uC_V: track 25.7 -> 36.9 mm
- net +3V3: track 43.0 -> 50.6 mm, vias 12 -> 16
- net /PyroPWR: track 6.46 -> 0.00 mm, vias 18 -> 16
- net /DeployV_Post_Diode: track 11.0 -> 5.19 mm, vias 7 -> 8
- net Net-(D18-A): track 48.5 -> 54.0 mm
- net /CHIP_PU: track 13.6 -> 9.64 mm
- net /SHNT_IN-: track 5.39 -> 8.27 mm
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Other:
- board size 44 x 58 mm -> 44 x 60 mm

Commit message: updated after rileys suggestions
Parts:
- moved G*** 9.50 mm to (117.6, 120.8)
- moved R35 3.26 mm to (130.8, 120.0)
- moved G*** 2.62 mm to (115.4, 82.8)
- moved R25 2.20 mm to (131.7, 117.8), turned to -90 degrees
- moved R24 2.17 mm to (131.7, 108.2), turned to -90 degrees
- moved C19 2.00 mm to (129.4, 118.6), turned to 0 degrees
- moved R28 1.83 mm to (130.8, 115.9)
- moved R29 1.72 mm to (130.7, 106.3)
- moved R22 1.50 mm to (130.7, 87.4)
- moved R34 1.01 mm to (129.8, 120.0)
- moved Q6 0.85 mm to (123.8, 122.9)
- moved Q5 0.57 mm to (118.0, 121.2)
- moved R46 0.42 mm to (110.0, 101.2)
- moved 16VLED2 0.42 mm to (141.5, 125.2)
- moved R45 0.38 mm to (111.9, 101.2)
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Routing:
- net /PyroPWR: track 0.00 -> 5.29 mm, vias 16 -> 13
- net /SHNT_IN-: track 8.27 -> 5.10 mm
- net /DeployV_Post_Diode: track 5.19 -> 7.96 mm, vias 8 -> 6
- net +3V3: track 50.6 -> 48.7 mm
- net /Nuke 0: track 7.48 -> 8.50 mm
- net /Nuke 2: track 22.2 -> 23.2 mm
- net /Nuke 3: track 28.4 -> 29.4 mm
- net /SHNT_IN+: track 3.48 -> 4.38 mm
- net /High side master switch/DGate: track 3.93 -> 4.57 mm
- net /CAN-: track 12.5 -> 12.0 mm
- net GND: vias 124 -> 133
- added copper zone on B.Cu, net +3V3
Other:
- board text added: "Designed By Electronics 2026"
- board text added: "FLINT & STEEL v4.0"
- board text removed: "Designed By Andrei Paduraru Electronics 2024"
- board text removed: "FLINT & STEEL v3.0"

Commit message: bomba
Other:
- board text added: "Designed By Andrei Paduraru Electronics 2024"
- board text added: "FLINT & STEEL v3.1"
- board text removed: "Designed By Electronics 2026"
- board text removed: "FLINT & STEEL v4.0"
Changed lines of the file:
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@@
 		)
 	)
-	(gr_text "FLINT & STEEL v4.0\n\n"
+	(gr_text "FLINT & STEEL v3.1\n\n"
 		(at 127.9 77.175 0)
 		(layer "B.SilkS")
@@
 		)
 	)
-	(gr_text "Designed By\nElectronics 2026"
-		(at 135.6 123.9 0)
+	(gr_text "Designed By\nAndrei Paduraru\nElectronics 2024"
+		(at 134.6 123 0)
 		(layer "B.SilkS")
 		(effects

Commit message: tidied up schematic and bom
Parts:
- C103: renamed from C3; value 0.1uF -> 100nF
- C105: renamed from C5; value 0.1uF -> 100nF
- C106: renamed from C6; value 0.1uF -> 100nF
- C108: renamed from C8; value 0.1uF -> 100nF
- C110: renamed from C10; value 0.1uF -> 100nF
- C111: renamed from C11; value 0.1uF -> 100nF
- C114: renamed from C19; value 0.1uF -> 100nF
- C115: renamed from C18; value 0.1uF -> 100nF
- C208: renamed from C27; value 0.1uF -> 100nF
- C301: renamed from C29; value 0.1uF -> 100nF
- C303: renamed from C28; value 0.1uF -> 100nF
- C304: renamed from C30; value 0.1uF -> 100nF
- D101: renamed from TXLED1; value GREEN_LED -> LED_GREEN
- D102: renamed from CANTXLED1; value GREEN_LED -> LED_GREEN
- D103: renamed from CANRXLED1; value ORANGE_LED -> LED_ORANGE
- D104: renamed from 3V3LED1; value BLUE_LED -> LED_BLUE
- D105: renamed from 16VLED2; value ORANGE_LED -> LED_ORANGE
- D106: renamed from 16VLED1; value RED_LED -> LED_RED
- D502: renamed from USBLED1; value WHITE_LED -> LED_WHITE
- D701: renamed from Firing1; value EMERALD_LED -> LED_GREEN
- D702: renamed from Firing2; value EMERALD_LED -> LED_GREEN
- D707: renamed from D6; value RED_LED -> LED_RED
- D708: renamed from D5; value RED_LED -> LED_RED
- D711: renamed from Firing4; value EMERALD_LED -> LED_GREEN
- D712: renamed from Firing3; value EMERALD_LED -> LED_GREEN
- D717: renamed from D9; value RED_LED -> LED_RED
- D718: renamed from D10; value RED_LED -> LED_RED
- L101: renamed from L1; value 2.0nH -> 2nH
- R101: renamed from R1; value 10K -> 10kΩ
- R102: renamed from R2; value 470 -> 470Ω
- R103: renamed from R7; value 1k -> 1kΩ
- R104: renamed from R30; value 1k -> 1kΩ
- R105: renamed from R3; value 10K -> 10kΩ
- R106: renamed from R4; value 470 -> 470Ω
- R107: renamed from R6; value 499 -> 499Ω
- R108: renamed from R40; value 3k -> 3kΩ
- R109: renamed from R36; value 3k -> 3kΩ
- R110: renamed from R33; value 2m -> 2mΩ
- R111: renamed from R47; value 10k -> 10kΩ
- R112: renamed from R34; value 10 -> 10Ω
- R113: renamed from R35; value 10 -> 10Ω
- R114: renamed from R31; value 3.3k -> 3.3kΩ
- R115: renamed from R32; value 3.3k -> 3.3kΩ
- R201: renamed from R14; value 10k -> 10kΩ
- R202: renamed from R15; value 14k -> 14kΩ
- R203: renamed from R16; value 56k -> 56kΩ
- R204: renamed from R17; value 10k -> 10kΩ
- R301: renamed from R5; value 10k -> 10kΩ
- R302: renamed from R37; value 100k -> 100kΩ
- R303: renamed from R38; value 5.1k -> 5.1kΩ
- R304: renamed from R39; value 4.22k -> 4.22kΩ
- R401: renamed from R41; value 10k -> 10kΩ
- R402: renamed from R42; value 10k -> 10kΩ
- R403: renamed from R43; value 10k -> 10kΩ
- R404: renamed from R44; value 10k -> 10kΩ
- R405: renamed from R45; value 10k -> 10kΩ
- R406: renamed from R46; value 10k -> 10kΩ
- R501: renamed from R11; value 5.1k -> 5.1kΩ
- R502: renamed from R12; value 5.1k -> 5.1kΩ
- R503: renamed from R13; value 5.1k -> 5.1kΩ
- R601: renamed from R8; value 0 -> 0Ω
- R602: renamed from R9; value 60 -> 60Ω
- R603: renamed from R10; value 60 -> 60Ω
- R701: renamed from R18; value 120 -> 120Ω
- R702: renamed from R19; value 120 -> 120Ω
- R703: renamed from R22; value 10K -> 10kΩ
- R704: renamed from R23; value 10K -> 10kΩ
- R705: renamed from R21; value 120 -> 120Ω
- R706: renamed from R20; value 120 -> 120Ω
- R707: renamed from R25; value 120 -> 120Ω
- R708: renamed from R24; value 120 -> 120Ω
- R709: renamed from R29; value 10K -> 10kΩ
- R710: renamed from R28; value 10K -> 10kΩ
- R711: renamed from R26; value 120 -> 120Ω
- R712: renamed from R27; value 120 -> 120Ω
- U203: renamed from U5; value SC4215 -> SC4215ASTRT
- Y101: renamed from Y1; value R940000171 -> 40MHz±10ppm; footprint iclr:Crystal_SMD_2016-4Pin_2.0x1.6mm -> Crystal:Crystal_SMD_2016-4Pin_2.0x1.6mm
- moved C112 0.11 mm to (123.2, 81.0)
- moved C113 0.11 mm to (119.2, 81.1)
- renumbered C1 to C101, C2 to C102, C4 to C104, C7 to C107, C9 to C109, C13 to C112, C14 to C113, C20 to C201, C21 to C202, C22 to C203, C23 to C204, C24 to C205, C25 to C206, C26 to C207, C12 to C302, C15 to C601, C16 to C602, C17 to C603, D19 to D301, D20 to D401, D2 to D501, D1 to D601, D15 to D703, D16 to D704, D7 to D705, D3 to D706, D14 to D709, D11 to D710, D17 to D713, D18 to D714, D4 to D715, D8 to D716, D12 to D719, D13 to D720, H1 to H101, H2 to H102, H3 to H103, H4 to H104, ENJUMPER1 to J101, BOOTJUMPER1 to J102, J1 to J103, J6 to J401, J2 to J501, J7 to J701, J3 to J702, J4 to J703, J5 to J704, JP1 to JP601, L2 to L102, L3 to L201, Q5 to Q301, Q6 to Q302, Q1 to Q701, Q2 to Q702, Q3 to Q703, Q4 to Q704, TP9 to TP101, TP10 to TP102, TP4 to TP103, TP3 to TP104, TP8 to TP201, TP6 to TP202, TP1 to TP501, TP2 to TP502, U1 to U101, U7 to U102, U3 to U201, U4 to U202, U8 to U301, U2 to U601, U6 to U701
