File: Hardware/power.kicad_sch (KiCad schematic)
At the start: 21 parts, among them U3 LM66200DRLR, U4 MAX77827AEFD+T, U5 SC4215

Commit message: schematic done? + footprints assigned
Parts:
- U3: footprint SOTFL50P160X60-8N -> iclr:SOTFL50P160X60-8N
Changed lines of the file:
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@@
       (effects (font (size 1.27 1.27)))
     )
-    (property "Footprint" "SOTFL50P160X60-8N" (at 76.2 34.29 0)
+    (property "Footprint" "iclr:SOTFL50P160X60-8N" (at 76.2 34.29 0)
       (effects (font (size 1.27 1.27)) (justify left) hide)
     )

Commit message: finished? (pre-review)
Parts:
- removed TP4, TP5, TP7: TestPoint, TestPoint:TestPoint_Pad_D1.5mm, symbol Connector:TestPoint
- TP6, TP8: footprint TestPoint:TestPoint_Pad_D1.5mm -> TestPoint:TestPoint_Pad_D1.0mm
Other:
- note removed: "Place close together. Bridge to bypass buck-boost"
- moved on the sheet: TP6
Changed lines of the file:
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@@
   (junction (at 166.37 52.07) (diameter 0) (color 0 0 0 0)
-  )
-  (junction (at 123.19 52.07) (diameter 0) (color 0 0 0 0)
   )
   (junction (at 240.03 60.96) (diameter 0) (color 0 0 0 0)
@@
     (stroke (width 0) (type default))
   )
-  (polyline (pts (xy 129.54 21.59) (xy 129.54 35.56))
-    (stroke (width 0) (type default))
-  )
   (wire (pts (xy 133.35 57.15) (xy 135.89 57.15))
     (stroke (width 0) (type default))
@@
     (stroke (width 0) (type default))
   )
-  (wire (pts (xy 123.19 52.07) (xy 128.27 52.07))
+  (wire (pts (xy 101.6 52.07) (xy 128.27 52.07))
     (stroke (width 0) (type default))
   )
@@
     (stroke (width 0) (type default))
   )
-  (wire (pts (xy 101.6 52.07) (xy 123.19 52.07))
-    (stroke (width 0) (type default))
-  )
   (wire (pts (xy 186.69 57.15) (xy 184.15 57.15))
     (stroke (width 0) (type default))
   )
-  (polyline (pts (xy 173.99 35.56) (xy 129.54 35.56))
-    (stroke (width 0) (type default))
-  )
-  (polyline (pts (xy 173.99 21.59) (xy 173.99 35.56))
-    (stroke (width 0) (type default))
-  )
   (wire (pts (xy 153.67 119.38) (xy 158.75 119.38))
     (stroke (width 0) (type default))
@@
     (stroke (width 0) (type default))
   )
-  (polyline (pts (xy 129.54 21.59) (xy 173.99 21.59))
-    (stroke (width 0) (type default))
-  )
   (wire (pts (xy 166.37 54.61) (xy 166.37 52.07))
     (stroke (width 0) (type default))
@@
   (wire (pts (xy 132.08 74.93) (xy 132.08 72.39))
     (stroke (width 0) (type default))
-  )
-  (text "Place close together.\nBridge to bypass buck-boost\n"
-    (at 137.16 20.32 0)
-    (effects (font (size 1.27 1.27)) (justify left bottom))
   )
   (text "Be extra careful in leaving this connected at a single point\n"
@@
     (effects (font (size 1.27 1.27)) (justify right bottom))
   )
-  (global_label "RBUS_uC_V" (shape input) (at 147.32 29.21 180) (fields_autoplaced)
-    (effects (font (size 1.27 1.27)) (justify right))
-    (property "Intersheetrefs" "${INTERSHEET_REFS}" (at 134.4729 29.1306 0)
-      (effects (font (size 1.27 1.27)) (justify right) hide)
-    )
-  )
   (global_label "RBUS_uC_V" (shape input) (at 90.17 39.37 0) (fields_autoplaced)
     (effects (font (size 1.27 1.27)) (justify left))
@@
     )
   )
-  (symbol (lib_id "power:+3.3V") (at 161.29 29.21 0) (unit 1)
-    (in_bom yes) (on_board yes) (dnp no) (fields_autoplaced)
-    (property "Reference" "#PWR043" (at 161.29 33.02 0)
-      (effects (font (size 1.27 1.27)) hide)
-    )
-    (property "Value" "+3.3V" (at 161.29 25.6342 0)
-      (effects (font (size 1.27 1.27)))
-    )
-    (property "Footprint" "" (at 161.29 29.21 0)
-      (effects (font (size 1.27 1.27)) hide)
-    )
-    (property "Datasheet" "" (at 161.29 29.21 0)
+  (symbol (lib_id "power:+3.3V") (at 195.1069 44.4136 0) (unit 1)
+    (in_bom yes) (on_board yes) (dnp no) (fields_autoplaced)
+    (property "Reference" "#PWR043" (at 195.1069 48.2236 0)
+      (effects (font (size 1.27 1.27)) hide)
+    )
+    (property "Value" "+3.3V" (at 195.1069 40.8378 0)
+      (effects (font (size 1.27 1.27)))
+    )
+    (property "Footprint" "" (at 195.1069 44.4136 0)
+      (effects (font (size 1.27 1.27)) hide)
+    )
+    (property "Datasheet" "" (at 195.1069 44.4136 0)
       (effects (font (size 1.27 1.27)) hide)
     )
@@
       (effects (font (size 1.27 1.27)) (justify left))
     )
-    (property "Footprint" "TestPoint:TestPoint_Pad_D1.5mm" (at 196.85 50.8 0)
+    (property "Footprint" "TestPoint:TestPoint_Pad_D1.0mm" (at 196.85 50.8 0)
       (effects (font (size 1.27 1.27)) hide)
     )
@@
     )
   )
-  (symbol (lib_id "Connector:TestPoint") (at 147.32 29.21 270) (unit 1)
-    (in_bom yes) (on_board yes) (dnp no)
-    (property "Reference" "TP5" (at 146.05 31.75 90)
-      (effects (font (size 1.27 1.27)) (justify left))
-    )
-    (property "Value" "TestPoint" (at 146.05 34.2869 90)
-      (effects (font (size 1.27 1.27)) (justify left))
-    )
-    (property "Footprint" "TestPoint:TestPoint_Pad_D1.5mm" (at 147.32 34.29 0)
-      (effects (font (size 1.27 1.27)) hide)
-    )
-    (property "Datasheet" "~" (at 147.32 34.29 0)
-      (effects (font (size 1.27 1.27)) hide)
-    )
-    (pin "1")
-    (instances
-      (project "flintandsteel"
-        (path "/7db990e4-92e1-4f99-b4d2-435bbec1ba83/48a413b4-b7c2-44ac-971c-583c31b73475"
-          (reference "TP5") (unit 1)
-        )
-      )
-    )
-  )
-  (symbol (lib_id "power:VBUS") (at 191.77 40.64 0) (unit 1)
-    (in_bom yes) (on_board yes) (dnp no) (fields_autoplaced)
-    (property "Reference" "#PWR046" (at 191.77 44.45 0)
-      (effects (font (size 1.27 1.27)) hide)
-    )
-    (property "Value" "VBUS" (at 191.77 37.0642 0)
-      (effects (font (size 1.27 1.27)))
-    )
-    (property "Footprint" "" (at 191.77 40.64 0)
-      (effects (font (size 1.27 1.27)) hide)
-    )
-    (property "Datasheet" "" (at 191.77 40.64 0)
-      (effects (font (size 1.27 1.27)) hide)
-    )
-    (pin "1")
-    (instances
-      (project "flintandsteel"
-        (path "/7db990e4-92e1-4f99-b4d2-435bbec1ba83/48a413b4-b7c2-44ac-971c-583c31b73475"
-          (reference "#PWR046") (unit 1)
-        )
-      )
-    )
-  )
   (symbol (lib_id "Device:C_Small") (at 184.15 54.61 0) (unit 1)
     (in_bom yes) (on_board yes) (dnp no)
@@
     )
   )
-  (symbol (lib_id "Connector:TestPoint") (at 123.19 52.07 0) (unit 1)
-    (in_bom yes) (on_board yes) (dnp no)
-    (property "Reference" "TP4" (at 121.92 45.72 0)
-      (effects (font (size 1.27 1.27)) (justify left))
-    )
-    (property "Value" "TestPoint" (at 121.92 43.1831 0)
-      (effects (font (size 1.27 1.27)) (justify left))
-    )
-    (property "Footprint" "TestPoint:TestPoint_Pad_D1.5mm" (at 128.27 52.07 0)
-      (effects (font (size 1.27 1.27)) hide)
-    )
-    (property "Datasheet" "~" (at 128.27 52.07 0)
-      (effects (font (size 1.27 1.27)) hide)
-    )
-    (pin "1")
-    (instances
-      (project "flintandsteel"
-        (path "/7db990e4-92e1-4f99-b4d2-435bbec1ba83/48a413b4-b7c2-44ac-971c-583c31b73475"
-          (reference "TP4") (unit 1)
-        )
-      )
-    )
-  )
   (symbol (lib_id "Device:R_Small") (at 240.03 64.77 0) (unit 1)
     (in_bom yes) (on_board yes) (dnp no)
@@
         (path "/7db990e4-92e1-4f99-b4d2-435bbec1ba83/48a413b4-b7c2-44ac-971c-583c31b73475"
           (reference "#PWR049") (unit 1)
-        )
-      )
-    )
-  )
-  (symbol (lib_id "Connector:TestPoint") (at 191.77 40.64 180) (unit 1)
-    (in_bom yes) (on_board yes) (dnp no)
-    (property "Reference" "TP7" (at 185.42 40.64 0)
-      (effects (font (size 1.27 1.27)) (justify left))
-    )
-    (property "Value" "TestPoint" (at 190.5 43.1769 0)
-      (effects (font (size 1.27 1.27)) (justify left))
-    )
-    (property "Footprint" "TestPoint:TestPoint_Pad_D1.5mm" (at 186.69 40.64 0)
-      (effects (font (size 1.27 1.27)) hide)
-    )
-    (property "Datasheet" "~" (at 186.69 40.64 0)
-      (effects (font (size 1.27 1.27)) hide)
-    )
-    (pin "1")
-    (instances
-      (project "flintandsteel"
-        (path "/7db990e4-92e1-4f99-b4d2-435bbec1ba83/48a413b4-b7c2-44ac-971c-583c31b73475"
-          (reference "TP7") (unit 1)
         )
       )
@@
     )
   )
-  (symbol (lib_id "Connector:TestPoint") (at 161.29 29.21 90) (unit 1)
-    (in_bom yes) (on_board yes) (dnp no)
-    (property "Reference" "TP6" (at 166.37 26.67 90)
-      (effects (font (size 1.27 1.27)))
-    )
-    (property "Value" "TestPoint" (at 169.291 28.7716 90)
-      (effects (font (size 1.27 1.27)))
-    )
-    (property "Footprint" "TestPoint:TestPoint_Pad_D1.5mm" (at 161.29 24.13 0)
-      (effects (font (size 1.27 1.27)) hide)
-    )
-    (property "Datasheet" "~" (at 161.29 24.13 0)
-      (effects (font (size 1.27 1.27)) hide)
-    )
+  (symbol (lib_id "Connector:TestPoint") (at 195.1069 44.4136 90) (unit 1)
+    (in_bom yes) (on_board yes) (dnp no)
+    (property "Reference" "TP6" (at 200.1869 41.8736 90)
+      (effects (font (size 1.27 1.27)))
+    )
+    (property "Value" "TestPoint" (at 203.1079 43.9752 90)
+      (effects (font (size 1.27 1.27)))
+    )
+    (property "Footprint" "TestPoint:TestPoint_Pad_D1.0mm" (at 195.1069 39.3336 0)
+      (effects (font (size 1.27 1.27)) hide)
+    )
+    (property "Datasheet" "~" (at 195.1069 39.3336 0)
+      (effects (font (size 1.27 1.27)) hide)
+    )
