File: Hardware/flintandsteel.kicad_sch (KiCad schematic)
At the start: 48 parts, among them J1 RBUS, U1 ESP32-S3, U7 INA219AxDCN, Y1 R940000171

Commit message: v2.1 ordering
Parts:
- removed C28: 0.1uF, Capacitor_SMD:C_0402_1005Metric, symbol Device:C_Small
- removed R30: 10k, Resistor_SMD:R_0402_1005Metric, symbol Device:R_Small
- removed R7: 124k, Resistor_SMD:R_0402_1005Metric, symbol Device:R_Small
- added TP3, TP4: TestPoint, TestPoint:TestPoint_Pad_D1.0mm, symbol Connector:TestPoint
- TXLED1: value TX_LED -> GREEN_LED
Connections:
- net SCL: now also TP3.1
- net SDA: now also TP4.1
Changed lines of the file:
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@@
   (junction (at 69.85 142.24) (diameter 0) (color 0 0 0 0)
   )
-  (junction (at 270.51 41.91) (diameter 0) (color 0 0 0 0)
-  )
   (junction (at 55.88 127) (diameter 0) (color 0 0 0 0)
   )
@@
   (junction (at 69.85 130.81) (diameter 0) (color 0 0 0 0)
   )
+  (junction (at 236.22 35.56) (diameter 0) (color 0 0 0 0)
+  )
   (junction (at 29.21 140.97) (diameter 0) (color 0 0 0 0)
   )
   (junction (at 16.51 170.18) (diameter 0) (color 0 0 0 0)
   )
-  (junction (at 274.32 46.99) (diameter 0) (color 0 0 0 0)
+  (junction (at 242.57 38.1) (diameter 0) (color 0 0 0 0)
   )
   (junction (at 270.51 33.02) (diameter 0) (color 0 0 0 0)
@@
     (stroke (width 0) (type default))
   )
+  (wire (pts (xy 236.22 35.56) (xy 240.03 35.56))
+    (stroke (width 0) (type default))
+  )
   (polyline (pts (xy 90.17 78.74) (xy 68.58 78.74))
     (stroke (width 0) (type default))
@@
     (stroke (width 0) (type default))
   )
-  (wire (pts (xy 270.51 41.91) (xy 274.32 41.91))
-    (stroke (width 0) (type default))
-  )
   (polyline (pts (xy 124.46 111.76) (xy 124.46 114.3))
     (stroke (width 0) (type default))
@@
     (stroke (width 0) (type default))
   )
-  (wire (pts (xy 231.14 35.56) (xy 240.03 35.56))
+  (wire (pts (xy 231.14 35.56) (xy 236.22 35.56))
     (stroke (width 0) (type default))
   )
@@
     (stroke (width 0) (type default))
   )
-  (wire (pts (xy 274.32 46.99) (xy 274.32 49.53))
-    (stroke (width 0) (type default))
-  )
   (wire (pts (xy 231.14 44.45) (xy 231.14 45.72))
     (stroke (width 0) (type default))
@@
     (stroke (width 0) (type default))
   )
-  (wire (pts (xy 270.51 46.99) (xy 274.32 46.99))
-    (stroke (width 0) (type default))
-  )
   (wire (pts (xy 20.32 135.89) (xy 29.21 135.89))
     (stroke (width 0) (type default))
@@
   )
   (wire (pts (xy 107.95 185.42) (xy 115.57 185.42))
-    (stroke (width 0) (type default))
-  )
-  (wire (pts (xy 265.43 41.91) (xy 270.51 41.91))
     (stroke (width 0) (type default))
   )
@@
     (effects (font (size 1.27 1.27)) (justify left bottom))
   )
-  (label "DeployV_SNS" (at 274.32 49.53 180) (fields_autoplaced)
-    (effects (font (size 1.27 1.27)) (justify right bottom))
-  )
   (label "BOOT" (at 68.58 165.1 180) (fields_autoplaced)
     (effects (font (size 1.27 1.27)) (justify right bottom))
@@
   (label "CAN_TX" (at 144.78 69.85 180) (fields_autoplaced)
     (effects (font (size 1.27 1.27)) (justify right bottom))
-  )
-  (label "DeployV" (at 265.43 41.91 0) (fields_autoplaced)
-    (effects (font (size 1.27 1.27)) (justify left bottom))
   )
   (label "TXD" (at 17.78 21.59 0) (fields_autoplaced)
@@
       (effects (font (size 1.27 1.27)))
     )
-    (property "Value" "TX_LED" (at 25.4 24.4856 0)
+    (property "Value" "GREEN_LED" (at 25.4 24.4856 0)
       (effects (font (size 1.27 1.27)))
     )
@@
   (symbol (lib_id "Device:LED_Small") (at 54.61 21.59 180) (unit 1)
     (in_bom yes) (on_board yes) (dnp no)
-    (property "Reference" "3V3LED1" (at 54.61 16.383 0)
-      (effects (font (size 1.27 1.27)))
-    )
-    (property "Value" "BLUE_LED" (at 54.61 18.6944 0)
+    (property "Reference" "3V3LED1" (at 55.88 16.51 0)
+      (effects (font (size 1.27 1.27)))
+    )
+    (property "Value" "BLUE_LED" (at 55.88 18.8214 0)
       (effects (font (size 1.27 1.27)))
     )
@@
     )
   )
-  (symbol (lib_id "Device:R_Small") (at 274.32 44.45 0) (unit 1)
-    (in_bom yes) (on_board yes) (dnp no) (fields_autoplaced)
-    (property "Reference" "R7" (at 276.86 43.815 0)
-      (effects (font (size 1.27 1.27)) (justify left))
-    )
-    (property "Value" "124k" (at 276.86 46.355 0)
-      (effects (font (size 1.27 1.27)) (justify left))
-    )
-    (property "Footprint" "Resistor_SMD:R_0402_1005Metric" (at 274.32 44.45 0)
-      (effects (font (size 1.27 1.27)) hide)
-    )
-    (property "Datasheet" "~" (at 274.32 44.45 0)
-      (effects (font (size 1.27 1.27)) hide)
-    )
-    (pin "1")
-    (pin "2")
-    (instances
-      (project "flintandsteel"
-        (path "/7db990e4-92e1-4f99-b4d2-435bbec1ba83"
-          (reference "R7") (unit 1)
+  (symbol (lib_id "Connector:TestPoint") (at 242.57 38.1 180) (unit 1)
+    (in_bom yes) (on_board yes) (dnp no)
+    (property "Reference" "TP3" (at 243.7384 42.8752 90)
+      (effects (font (size 1.27 1.27)) (justify left))
+    )
+    (property "Value" "TestPoint" (at 241.427 42.8752 90)
+      (effects (font (size 1.27 1.27)) (justify left))
+    )
+    (property "Footprint" "TestPoint:TestPoint_Pad_D1.0mm" (at 237.49 38.1 0)
+      (effects (font (size 1.27 1.27)) hide)
+    )
+    (property "Datasheet" "~" (at 237.49 38.1 0)
+      (effects (font (size 1.27 1.27)) hide)
+    )
+    (pin "1")
+    (instances
+      (project "flintandsteel"
+        (path "/7db990e4-92e1-4f99-b4d2-435bbec1ba83"
+          (reference "TP3") (unit 1)
         )
       )
@@
     )
   )
-  (symbol (lib_id "power:GND") (at 274.32 54.61 0) (unit 1)
-    (in_bom yes) (on_board yes) (dnp no)
-    (property "Reference" "#PWR015" (at 274.32 60.96 0)
-      (effects (font (size 1.27 1.27)) hide)
-    )
-    (property "Value" "GND" (at 274.447 57.8612 90)
-      (effects (font (size 1.27 1.27)) (justify right))
-    )
-    (property "Footprint" "" (at 274.32 54.61 0)
-      (effects (font (size 1.27 1.27)) hide)
-    )
-    (property "Datasheet" "" (at 274.32 54.61 0)
-      (effects (font (size 1.27 1.27)) hide)
-    )
-    (pin "1")
-    (instances
-      (project "flintandsteel"
-        (path "/7db990e4-92e1-4f99-b4d2-435bbec1ba83"
-          (reference "#PWR015") (unit 1)
-        )
-      )
-    )
-  )
   (symbol (lib_id "Device:C_Small") (at 50.8 129.54 0) (unit 1)
     (in_bom yes) (on_board yes) (dnp no)
@@
         (path "/7db990e4-92e1-4f99-b4d2-435bbec1ba83"
           (reference "#PWR014") (unit 1)
-        )
-      )
-    )
-  )
-  (symbol (lib_id "Device:R_Small") (at 274.32 52.07 0) (unit 1)
-    (in_bom yes) (on_board yes) (dnp no) (fields_autoplaced)
-    (property "Reference" "R30" (at 276.86 51.435 0)
-      (effects (font (size 1.27 1.27)) (justify left))
-    )
-    (property "Value" "10k" (at 276.86 53.975 0)
-      (effects (font (size 1.27 1.27)) (justify left))
-    )
-    (property "Footprint" "Resistor_SMD:R_0402_1005Metric" (at 274.32 52.07 0)
-      (effects (font (size 1.27 1.27)) hide)
-    )
-    (property "Datasheet" "~" (at 274.32 52.07 0)
-      (effects (font (size 1.27 1.27)) hide)
-    )
-    (pin "1")
-    (pin "2")
-    (instances
-      (project "flintandsteel"
-        (path "/7db990e4-92e1-4f99-b4d2-435bbec1ba83"
-          (reference "R30") (unit 1)
         )
       )
@@
     (in_bom yes) (on_board yes) (dnp no)
     (property "Reference" "R31" (at 234.95 30.48 0)
-      (effects (font (size 1.27 1.27)) (justify left))
+      (effects (font (size 1.27 1.27)) (justify left) hide)
     )
     (property "Value" "3.3k" (at 234.95 33.02 0)
-      (effects (font (size 1.27 1.27)) (justify left))
+      (effects (font (size 1.27 1.27)) (justify left) hide)
     )
     (property "Footprint" "Resistor_SMD:R_0402_1005Metric" (at 240.03 33.02 0)
@@
     )
   )
-  (symbol (lib_id "Device:C_Small") (at 270.51 44.45 0) (unit 1)
-    (in_bom yes) (on_board yes) (dnp no)
-    (property "Reference" "C28" (at 262.89 43.18 0)
-      (effects (font (size 1.27 1.27)) (justify left))
-    )
-    (property "Value" "0.1uF" (at 262.89 45.72 0)
-      (effects (font (size 1.27 1.27)) (justify left))
-    )
-    (property "Footprint" "Capacitor_SMD:C_0402_1005Metric" (at 270.51 44.45 0)
-      (effects (font (size 1.27 1.27)) hide)
-    )
-    (property "Datasheet" "~" (at 270.51 44.45 0)
-      (effects (font (size 1.27 1.27)) hide)
-    )
-    (pin "1")
-    (pin "2")
-    (instances
-      (project "flintandsteel"
-        (path "/7db990e4-92e1-4f99-b4d2-435bbec1ba83"
-          (reference "C28") (unit 1)
-        )
-      )
-    )
-  )
   (symbol (lib_id "power:GND") (at 50.8 62.23 0) (unit 1)
     (in_bom yes) (on_board yes) (dnp no)
@@
         )
       )
+    )
+  )
+  (symbol (lib_id "Connector:TestPoint") (at 236.22 35.56 0) (unit 1)
+    (in_bom yes) (on_board yes) (dnp no)
+    (property "Reference" "TP4" (at 235.0516 30.7848 90)
+      (effects (font (size 1.27 1.27)) (justify left))
+    )
+    (property "Value" "TestPoint" (at 237.363 30.7848 90)
+      (effects (font (size 1.27 1.27)) (justify left))
+    )
+    (property "Footprint" "TestPoint:TestPoint_Pad_D1.0mm" (at 241.3 35.56 0)
+      (effects (font (size 1.27 1.27)) hide)
+    )
+    (property "Datasheet" "~" (at 241.3 35.56 0)
+      (effects (font (size 1.27 1.27)) hide)
+    )
+    (pin "1")
+    (instances
+      (project "flintandsteel"
+        (path "/7db990e4-92e1-4f99-b4d2-435bbec1ba83"
+          (reference "TP4") (unit 1)
+        )
+      )
