File: Hardware/GPIO.kicad_sch (KiCad schematic)
At the start: 8 parts, among them J6 GPIO Breakout

Commit message: tidied up schematic and bom
Parts:
- R401: renamed from R41; value 10k -> 10kΩ
- R402: renamed from R42; value 10k -> 10kΩ
- R403: renamed from R43; value 10k -> 10kΩ
- R404: renamed from R44; value 10k -> 10kΩ
- R405: renamed from R45; value 10k -> 10kΩ
- R406: renamed from R46; value 10k -> 10kΩ
- renumbered D20 to D401, J6 to J401
Changed lines of the file:
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@@
 		(on_board yes)
 		(dnp yes)
-		(property "Reference" "R41"
+		(property "Reference" "R401"
 			(at 141.1986 128.3716 0)
 			(effects
@@
 			)
 		)
-		(property "Value" "10k"
+		(property "Value" "10kΩ"
 			(at 141.1986 130.683 0)
 			(effects
@@
 			(project "flintandsteel"
 				(path "/7db990e4-92e1-4f99-b4d2-435bbec1ba83/acf6a9c3-1e4d-4cfc-afe3-1c8d949fad1a"
-					(reference "R41")
+					(reference "R401")
 					(unit 1)
 				)
@@
 		(on_board yes)
 		(dnp yes)
-		(property "Reference" "R45"
+		(property "Reference" "R405"
 			(at 169.1386 128.3716 0)
 			(effects
@@
 			)
 		)
-		(property "Value" "10k"
+		(property "Value" "10kΩ"
 			(at 169.1386 130.683 0)
 			(effects
@@
 			(project "flintandsteel"
 				(path "/7db990e4-92e1-4f99-b4d2-435bbec1ba83/acf6a9c3-1e4d-4cfc-afe3-1c8d949fad1a"
-					(reference "R45")
+					(reference "R405")
 					(unit 1)
 				)
@@
 		(on_board yes)
 		(dnp no)
-		(property "Reference" "#PWR078"
+		(property "Reference" "#PWR0401"
 			(at 90.17 95.25 0)
 			(effects
@@
 			(project "flintandsteel"
 				(path "/7db990e4-92e1-4f99-b4d2-435bbec1ba83/acf6a9c3-1e4d-4cfc-afe3-1c8d949fad1a"
-					(reference "#PWR078")
+					(reference "#PWR0401")
 					(unit 1)
 				)
@@
 		(dnp no)
 		(fields_autoplaced yes)
-		(property "Reference" "D20"
+		(property "Reference" "D401"
 			(at 118.11 78.74 0)
 			(effects
@@
 			(project "flintandsteel"
 				(path "/7db990e4-92e1-4f99-b4d2-435bbec1ba83/acf6a9c3-1e4d-4cfc-afe3-1c8d949fad1a"
-					(reference "D20")
+					(reference "D401")
 					(unit 1)
 				)
@@
 		(dnp no)
 		(fields_autoplaced yes)
-		(property "Reference" "#PWR0101"
+		(property "Reference" "#PWR0402"
 			(at 157.48 130.81 0)
 			(effects
@@
 			(project "flintandsteel"
 				(path "/7db990e4-92e1-4f99-b4d2-435bbec1ba83/acf6a9c3-1e4d-4cfc-afe3-1c8d949fad1a"
-					(reference "#PWR0101")
+					(reference "#PWR0402")
 					(unit 1)
 				)
@@
 		(on_board yes)
 		(dnp no)
-		(property "Reference" "J6"
+		(property "Reference" "J401"
 			(at 184.15 109.22 90)
 			(effects
@@
 			(project "flintandsteel"
 				(path "/7db990e4-92e1-4f99-b4d2-435bbec1ba83/acf6a9c3-1e4d-4cfc-afe3-1c8d949fad1a"
-					(reference "J6")
+					(reference "J401")
 					(unit 1)
 				)
@@
 		(on_board yes)
 		(dnp yes)
-		(property "Reference" "R42"
+		(property "Reference" "R402"
 			(at 147.5486 128.3716 0)
 			(effects
@@
 			)
 		)
-		(property "Value" "10k"
+		(property "Value" "10kΩ"
 			(at 147.5486 130.683 0)
 			(effects
@@
 			(project "flintandsteel"
 				(path "/7db990e4-92e1-4f99-b4d2-435bbec1ba83/acf6a9c3-1e4d-4cfc-afe3-1c8d949fad1a"
-					(reference "R42")
+					(reference "R402")
 					(unit 1)
 				)
@@
 		(on_board yes)
 		(dnp yes)
-		(property "Reference" "R43"
+		(property "Reference" "R403"
 			(at 155.1686 128.3716 0)
 			(effects
@@
 			)
 		)
-		(property "Value" "10k"
+		(property "Value" "10kΩ"
 			(at 155.1686 130.683 0)
 			(effects
@@
 			(project "flintandsteel"
 				(path "/7db990e4-92e1-4f99-b4d2-435bbec1ba83/acf6a9c3-1e4d-4cfc-afe3-1c8d949fad1a"
-					(reference "R43")
+					(reference "R403")
 					(unit 1)
 				)
@@
 		(on_board yes)
 		(dnp yes)
-		(property "Reference" "R46"
+		(property "Reference" "R406"
 			(at 176.7586 128.3716 0)
 			(effects
@@
 			)
 		)
-		(property "Value" "10k"
+		(property "Value" "10kΩ"
 			(at 176.7586 130.683 0)
 			(effects
@@
 			(project "flintandsteel"
 				(path "/7db990e4-92e1-4f99-b4d2-435bbec1ba83/acf6a9c3-1e4d-4cfc-afe3-1c8d949fad1a"
-					(reference "R46")
+					(reference "R406")
 					(unit 1)
 				)
@@
 		(dnp no)
 		(fields_autoplaced yes)
-		(property "Reference" "#PWR080"
+		(property "Reference" "#PWR0403"
 			(at 170.18 95.25 0)
 			(effects
@@
 			(project "flintandsteel"
 				(path "/7db990e4-92e1-4f99-b4d2-435bbec1ba83/acf6a9c3-1e4d-4cfc-afe3-1c8d949fad1a"
-					(reference "#PWR080")
+					(reference "#PWR0403")
 					(unit 1)
 				)
@@
 		(dnp no)
 		(fields_autoplaced yes)
-		(property "Reference" "#PWR079"
+		(property "Reference" "#PWR0404"
 			(at 180.34 105.41 0)
 			(effects
@@
 			(project "flintandsteel"
 				(path "/7db990e4-92e1-4f99-b4d2-435bbec1ba83/acf6a9c3-1e4d-4cfc-afe3-1c8d949fad1a"
-					(reference "#PWR079")
+					(reference "#PWR0404")
 					(unit 1)
 				)
@@
 		(on_board yes)
 		(dnp yes)
-		(property "Reference" "R44"
+		(property "Reference" "R404"
 			(at 162.7886 128.3716 0)
 			(effects
@@
 			)
 		)
-		(property "Value" "10k"
+		(property "Value" "10kΩ"
 			(at 162.7886 130.683 0)
 			(effects
@@
 			(project "flintandsteel"
 				(path "/7db990e4-92e1-4f99-b4d2-435bbec1ba83/acf6a9c3-1e4d-4cfc-afe3-1c8d949fad1a"
-					(reference "R44")
-					(unit 1)
-				)
+					(reference "R404")
+					(unit 1)
+				)
