File: Hardware/ematch.kicad_sch (KiCad schematic)
At the start: 33 parts, among them J3 Conn_01x02_Male, J4 Conn_01x02_Male, J5 Conn_01x02_Male, J6 Conn_01x02_Male, Q1 BUK9M11-40EX, Q2 BUK9M11-40EX, Q3 BUK9M11-40EX, Q4 BUK9M11-40EX, U6 LTV-247

Commit message: v3 hardware I guess
Parts:
- removed Q1, Q2, Q3, Q4: BUK9M11-40EX, Package_TO_SOT_SMD:LFPAK33, symbol Transistor_FET:BUK9M11-40EX
- added D11, D12, D13, D14: S-102T, iclr:SODFL3516X70N, symbol iclr:S-102T
- added D15, D16, D17, D18: V8PAM10S-M3/I, iclr:V8PAM10SM3I, symbol Device:D_Schottky_Small_Filled
- added Q1, Q2, Q3, Q4: BSZ025N04LS, iclr:BSZ025N04LS, symbol iclr:BSZ025N04LS
- R22, R23, R28, R29: value 10k -> 10K; footprint Resistor_SMD:R_0603_1608Metric -> Resistor_SMD:R_0402_1005Metric
Connections:
- net Nuke 4 is gone; now on net Nuke 3: Firing4.2 (A)
- net +3V3: now also U6.10, U6.12, U6.14, U6.16; no longer U6.10, U6.12, U6.14, U6.16
- net Cont1: now also R21.1, U6.11; no longer R20.1, U6.15
- net Cont2: now also R26.1, U6.13; no longer R21.1, U6.13
- net Cont3: now also R27.1, U6.15; no longer R26.1, U6.11
- net DeployPWR: now also D15.1 (K), D16.1 (K), D17.1 (K), D18.1 (K)
- net GND: now also D11.1 (K), D12.1 (K), D13.1 (K), D14.1 (K), Q1.1 (S), Q1.2 (S), Q1.3 (S), Q1.A1 (S), Q2.1 (S), Q2.2 (S), Q2.3 (S), Q2.A1 (S), Q3.1 (S), Q3.2 (S), Q3.3 (S), Q3.A1 (S), Q4.1 (S), Q4.2 (S), Q4.3 (S), Q4.A1 (S)
- net Nuke 1: now also Firing2.2 (A), R23.1, Q2.4 (G); no longer Firing1.2 (A)
- net Nuke 2: now also Firing3.2 (A), R29.1, Q3.4 (G); no longer Firing2.2 (A)
- net Nuke 3: now also R28.1, Q4.4 (G); no longer Firing3.2 (A)
- net at D3.1 (A), D3.2 (A), J3.2 (Pin_2): now also U6.7, D16.2 (A); no longer U6.1
- net at D3.3 (K): now also Q1.5 (D), Q1.6 (D), Q1.7 (D), Q1.8 (D), Q1.A5 (D)
- net at D7.3 (K): now also Q2.5 (D), Q2.6 (D), Q2.7 (D), Q2.8 (D), Q2.A5 (D)
- net at D7.1 (A), D7.2 (A), J4.2 (Pin_2): now also U6.5, D15.2 (A); no longer U6.3
- net at D8.1 (A), D8.2 (A), J6.2 (Pin_2): now also U6.1, D18.2 (A); no longer U6.7
- net at D4.1 (A), D4.2 (A), J5.2 (Pin_2): now also U6.3, D17.2 (A); no longer U6.5
- net at D4.3 (K): now also Q3.5 (D), Q3.6 (D), Q3.7 (D), Q3.8 (D), Q3.A5 (D)
- net Nuke 0: now reaches R22.1
- net Nuke 0: now also Firing1.2 (A), Q1.4 (G); no longer U6.2
- net at D8.3 (K): now also Q4.5 (D), Q4.6 (D), Q4.7 (D), Q4.8 (D), Q4.A5 (D)
- removed net Cont4: R27.1, U6.9
- new net: D12.2 (A), U6.4
- new net: D13.2 (A), U6.2
- new net: D11.2 (A), U6.8
- new net: D14.2 (A), U6.6
- new net Cont0: R20.1, U6.9
Other:
- note added: "+"
- note added: "-"

Commit message: files
Parts:
- removed J3, J4, J5, J6: Conn_01x02_Male, TerminalBlock_Phoenix:TerminalBlock_Phoenix_PT-1,5-2-3.5-H_1x02_P3.50mm_Horizontal, symbol Connector:Conn_01x02_Male
- added J3, J4, J5, J7: 1723103102, iclr:CONN_1723102000_02_MOL, symbol ICLR_HW:1723103102
Connections:
- net DeployPWR: now also J3.1, J4.1, J5.1, J7.1
- net at D16.2 (A), D3.1 (A), D3.2 (A)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: now also J3.2
- net at D18.2 (A), D8.1 (A), D8.2 (A)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: now also J5.2
- net at D15.2 (A), D7.1 (A), D7.2 (A)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: now also J7.2
- net at D17.2 (A), D4.1 (A), D4.2 (A)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: now also J4.2

Commit message: tidied up schematic and bom
Parts:
- D701: renamed from Firing1; value EMERALD_LED -> LED_GREEN
- D702: renamed from Firing2; value EMERALD_LED -> LED_GREEN
- D707: renamed from D6; value RED_LED -> LED_RED
- D708: renamed from D5; value RED_LED -> LED_RED
- D711: renamed from Firing4; value EMERALD_LED -> LED_GREEN
- D712: renamed from Firing3; value EMERALD_LED -> LED_GREEN
- D717: renamed from D9; value RED_LED -> LED_RED
- D718: renamed from D10; value RED_LED -> LED_RED
- R701: renamed from R18; value 120 -> 120Ω
- R702: renamed from R19; value 120 -> 120Ω
- R703: renamed from R22; value 10K -> 10kΩ
- R704: renamed from R23; value 10K -> 10kΩ
- R705: renamed from R21; value 120 -> 120Ω
- R706: renamed from R20; value 120 -> 120Ω
- R707: renamed from R25; value 120 -> 120Ω
- R708: renamed from R24; value 120 -> 120Ω
- R709: renamed from R29; value 10K -> 10kΩ
- R710: renamed from R28; value 10K -> 10kΩ
- R711: renamed from R26; value 120 -> 120Ω
- R712: renamed from R27; value 120 -> 120Ω
- renumbered D15 to D703, D16 to D704, D7 to D705, D3 to D706, D14 to D709, D11 to D710, D17 to D713, D18 to D714, D4 to D715, D8 to D716, D12 to D719, D13 to D720, J7 to J701, J3 to J702, J4 to J703, J5 to J704, Q1 to Q701, Q2 to Q702, Q3 to Q703, Q4 to Q704, U6 to U701
